File: circuit/Viper/ZRaiderViper.kicad_sch (KiCad schematic)
At the start: 29 parts, among them J1 DE9_Socket, J2 DE9_Socket, SW1 TRIGGER, SW10 DOWN, SW11 LEFT, SW2 SW_Push, SW3 SW_Push, SW4 UP, SW5 DOWN, SW6 LEFT, SW7 RIGHT, SW8 RIGHT, SW9 UP

Commit message: updating from Raider
Parts:
- added R4, R5: 300, Resistor_SMD:R_0805_2012Metric_Pad1.20x1.40mm_HandSolder, symbol Device:R_US
- SW2: value SW_Push -> TRIGGER
Connections:
- net at A1.19 (A0), S1.VR2_2: now also C1.2; no longer C1.1
- net at A1.29 (GND), A1.4 (GND), J1.8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: now also C1.1, C2.1, C3.1, C4.1; no longer C1.2, C2.2, C3.2, C4.2
- net at D1.2 (A): now also R5.2; no longer A1.7 (D4)
- net at D2.2 (A): now also R4.1; no longer A1.6 (D3)
- net at A1.21 (A2), S2.VR2_2: now also C3.2; no longer C3.1
- net at A1.20 (A1), S1.VR1_2: now also C2.2; no longer C2.1
- net at A1.22 (A3), S2.VR1_2: now also C4.2; no longer C4.1
- new net: A1.7 (D4), R5.1
- new net: A1.6 (D3), R4.2
- no-connect marks 8 -> 24
Other:
- moved on the sheet: C1, C2, C3, C4

Commit message: adding resistors to 2nd thumbstick output
Parts:
- added R6, R7: 300, Resistor_SMD:R_0805_2012Metric_Pad1.20x1.40mm_HandSolder, symbol Device:R_US
- SW3: value SW_Push -> Calibrate
Connections:
- net at D4.2 (A): now also R7.1; no longer A1.8 (D5)
- net at A1.5 (D2): now also R6.1; no longer D3.2 (A)
- new net: D3.2 (A), R6.2
- new net: A1.8 (D5), R7.2
- no-connect marks 24 -> 27
Changed lines of the file:
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@@
 	)
 	(no_connect
+		(at 153.67 191.77)
+	)
+	(no_connect
 		(at 179.07 143.51)
 	)
@@
 	)
 	(no_connect
+		(at 274.32 148.59)
+	)
+	(no_connect
 		(at 153.67 143.51)
 	)
@@
 	)
 	(no_connect
+		(at 153.67 148.59)
+	)
+	(no_connect
 		(at 210.82 194.31)
 	)
@@
 	(wire
 		(pts
-			(xy 265.43 233.68) (xy 176.53 233.68)
+			(xy 265.43 233.68) (xy 247.65 233.68)
 		)
 		(stroke
@@
 	(wire
 		(pts
+			(xy 240.03 233.68) (xy 176.53 233.68)
+		)
+		(stroke
+			(width 0)
+			(type default)
+		)
+	)
+	(wire
+		(pts
 			(xy 130.81 78.74) (xy 130.81 123.19)
 		)
@@
 	(wire
 		(pts
-			(xy 251.46 229.87) (xy 170.18 229.87)
+			(xy 251.46 229.87) (xy 238.76 229.87)
 		)
 		(stroke
@@
 	(wire
 		(pts
+			(xy 231.14 229.87) (xy 170.18 229.87)
+		)
+		(stroke
+			(width 0)
+			(type default)
+		)
+	)
+	(wire
+		(pts
 			(xy 133.35 191.77) (xy 151.13 191.77)
 		)
@@
 	)
 	(symbol
+		(lib_id "Device:R_US")
+		(at 234.95 229.87 90)
+		(unit 1)
+		(body_style 1)
+		(exclude_from_sim no)
+		(in_bom yes)
+		(on_board yes)
+		(in_pos_files yes)
+		(dnp no)
+		(property "Reference" "R6"
+			(at 235.966 224.79 90)
+			(show_name no)
+			(do_not_autoplace no)
+			(effects
+				(font
+					(size 1.27 1.27)
+				)
+				(justify left)
+			)
+		)
+		(property "Value" "300"
+			(at 236.2199 227.33 90)
+			(show_name no)
+			(do_not_autoplace no)
+			(effects
+				(font
+					(size 1.27 1.27)
+				)
+				(justify left)
+			)
+		)
+		(property "Footprint" "Resistor_SMD:R_0805_2012Metric_Pad1.20x1.40mm_HandSolder"
+			(at 235.204 228.854 90)
+			(hide yes)
+			(show_name no)
+			(do_not_autoplace no)
+			(effects
+				(font
+					(size 1.27 1.27)
+				)
+			)
+		)
+		(property "Datasheet" ""
+			(at 234.95 229.87 0)
+			(hide yes)
+			(show_name no)
+			(do_not_autoplace no)
+			(effects
+				(font
+					(size 1.27 1.27)
+				)
+			)
+		)
+		(property "Description" "Resistor, US symbol"
+			(at 234.95 229.87 0)
+			(hide yes)
+			(show_name no)
+			(do_not_autoplace no)
+			(effects
+				(font
+					(size 1.27 1.27)
+				)
+			)
+		)
+		(pin "1"
+		)
+		(pin "2"
+		)
+		(instances
+			(project "ZRaiderViper"
+				(path "/cee3fad8-cd38-4e35-ae79-7b381e15c120"
+					(reference "R6")
+					(unit 1)
+				)
+			)
+		)
+	)
+	(symbol
 		(lib_id "RKJXV122400R:RKJXV122400R")
 		(at 287.02 143.51 0)
@@
 			)
 		)
-		(property "Value" "SW_Push"
+		(property "Value" "Calibrate"
 			(at 146.05 207.01 0)
 			(show_name no)
@@
 					(unit 1)
 				)
+			)
+		)
+	)
+	(symbol
+		(lib_id "Device:R_US")
+		(at 243.84 233.68 270)
+		(unit 1)
+		(body_style 1)
+		(exclude_from_sim no)
+		(in_bom yes)
+		(on_board yes)
+		(in_pos_files yes)
+		(dnp no)
+		(property "Reference" "R7"
+			(at 243.84 235.458 90)
+			(show_name no)
+			(do_not_autoplace no)
+			(effects
+				(font
+					(size 1.27 1.27)
+				)
+			)
+		)
+		(property "Value" "300"
+			(at 243.586 237.49 90)
+			(show_name no)
+			(do_not_autoplace no)
+			(effects
+				(font
+					(size 1.27 1.27)
+				)
+			)
+		)
+		(property "Footprint" "Resistor_SMD:R_0805_2012Metric_Pad1.20x1.40mm_HandSolder"
+			(at 243.586 234.696 90)
+			(hide yes)
+			(show_name no)
+			(do_not_autoplace no)
+			(effects
+				(font
+					(size 1.27 1.27)
+				)
+			)
+		)
+		(property "Datasheet" ""
+			(at 243.84 233.68 0)
+			(hide yes)
+			(show_name no)
+			(do_not_autoplace no)
+			(effects
+				(font
+					(size 1.27 1.27)
+				)
+			)
+		)
+		(property "Description" "Resistor, US symbol"
+			(at 243.84 233.68 0)
+			(hide yes)
+			(show_name no)
+			(do_not_autoplace no)
+			(effects
+				(font
+					(size 1.27 1.27)
+				)
+			)
+		)
+		(pin "1"
+		)
+		(pin "2"
+		)
+		(instances
+			(project "ZRaiderViper"
+				(path "/cee3fad8-cd38-4e35-ae79-7b381e15c120"
+					(reference "R7")
+					(unit 1)
+				)

Commit message: fixing 300 resistors. updating labels
Parts:
- SW1: value TRIGGER -> TRIGGER_1
- SW10: value DOWN -> DOWN_2
- SW11: value LEFT -> LEFT_2
- SW2: value TRIGGER -> TRIGGER_2
- SW4: value UP -> UP_1
- SW5: value DOWN -> DOWN_1
- SW6: value LEFT -> LEFT_1
- SW7: value RIGHT -> RIGHT_1
- SW8: value RIGHT -> RIGHT_2
- SW9: value UP -> UP_2
Connections:
- net at A1.27 (+5V), D5.1 (K), R3.1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: now also S2.VR1_1, S2.VR2_1
- now unconnected: J2.7
- no-connect marks 27 -> 26
Other:
- moved on the sheet: S2A, S2B, S2C

Commit message: Fixing resistor val.
Parts:
- R4, R5, R6, R7: value 300 -> 330
Connections:
- no-connect marks 26 -> 27
Changed lines of the file:
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@@
 	)
 	(no_connect
+		(at 252.73 77.47)
+	)
+	(no_connect
 		(at 210.82 209.55)
 	)
@@
 			)
 		)
-		(property "Value" "300"
+		(property "Value" "330"
 			(at 237.998 227.33 90)
 			(show_name no)
@@
 			)
 		)
-		(property "Value" "300"
+		(property "Value" "330"
 			(at 163.576 198.12 90)
 			(show_name no)
@@
 			)
 		)
-		(property "Value" "300"
+		(property "Value" "330"
 			(at 156.2099 189.23 90)
 			(show_name no)
@@
 			)
 		)
-		(property "Value" "300"
+		(property "Value" "330"
 			(at 243.586 237.49 90)
 			(show_name no)

Commit message: working on viper PCB layout
Changed lines of the file:
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@@
+	)
+	(junction
+		(at 162.56 127)
+		(diameter 0)
+		(color 0 0 0 0)
+	)
+	(junction
+		(at 128.27 127)
+		(diameter 0)
+		(color 0 0 0 0)
 	)
 	(junction
@@
 	)
 	(junction
-		(at 128.27 129.54)
-		(diameter 0)
-		(color 0 0 0 0)
-	)
-	(junction
 		(at 289.56 121.92)
 		(diameter 0)
@@
 	(wire
 		(pts
+			(xy 162.56 127) (xy 257.81 127)
+		)
+		(stroke
+			(width 0)
+			(type default)
+		)
+	)
+	(wire
+		(pts
 			(xy 245.11 81.28) (xy 279.4 81.28)
 		)
@@
 	(wire
 		(pts
+			(xy 128.27 127) (xy 128.27 165.1)
+		)
+		(stroke
+			(width 0)
+			(type default)
+		)
+	)
+	(wire
+		(pts
 			(xy 124.46 187.96) (xy 124.46 182.88)
 		)
@@
 	(wire
 		(pts
-			(xy 128.27 78.74) (xy 128.27 129.54)
+			(xy 128.27 78.74) (xy 128.27 127)
 		)
 		(stroke
@@
 	(wire
 		(pts
-			(xy 128.27 129.54) (xy 128.27 165.1)
-		)
-		(stroke
-			(width 0)
-			(type default)
-		)
-	)
-	(wire
-		(pts
 			(xy 251.46 179.07) (xy 251.46 172.72)
 		)
@@
 	(wire
 		(pts
-			(xy 162.56 123.19) (xy 162.56 129.54)
+			(xy 162.56 123.19) (xy 162.56 127)
 		)
 		(stroke
@@
 	(wire
 		(pts
-			(xy 162.56 129.54) (xy 128.27 129.54)
-		)
-		(stroke
+			(xy 162.56 127) (xy 128.27 127)
+		)
+		(stroke
