File: circuit/Viper/ZRaiderViper.kicad_pcb (KiCad board)
At the start: 2 copper layers, 168 x 102 mm, 29 parts, among them J1 DE9_Socket, J2 DE9_Socket, SW1 SW_Push, SW10 SW_Push, SW11 SW_Push, SW2 SW_Push, SW3 SW_Push, SW4 SW_Push, SW5 SW_Push, SW6 SW_Push, SW7 SW_Push, SW8 SW_Push, SW9 SW_Push

Commit message: fixing 300 resistors. updating labels
Parts:
- added R4: 300, Resistor_SMD:R_0805_2012Metric_Pad1.20x1.40mm_HandSolder, F.Cu at (1.88, 0.97)
- added R5: 300, Resistor_SMD:R_0805_2012Metric_Pad1.20x1.40mm_HandSolder, F.Cu at (1.88, 3.92)
- SW1, SW2: value SW_Push -> TRIGGER
- SW10, SW5: value SW_Push -> DOWN
- SW11, SW6: value SW_Push -> LEFT
- SW4, SW9: value SW_Push -> UP
- SW7, SW8: value SW_Push -> RIGHT
Connections:
- A1 pad 12: Net-(A1-D9) -> unconnected-(A1-D9-Pad12)
- A1 pad 27: unconnected-(A1-+5V-Pad27) -> Net-(A1-+5V)
- A1 pad 5: unconnected-(A1-D2-Pad5) -> Net-(A1-D2)
- A1 pad 8: unconnected-(A1-D5-Pad8) -> Net-(A1-D5)
- C1 pad 1: Net-(A1-A0) -> Net-(A1-GND-Pad29)
- C1 pad 2: Net-(A1-GND-Pad29) -> Net-(A1-A0)
- C2 pad 1: Net-(A1-A1) -> Net-(A1-GND-Pad29)
- C2 pad 2: Net-(A1-GND-Pad29) -> Net-(A1-A1)
- C3 pad 1: Net-(A1-A2) -> Net-(A1-GND-Pad29)
- C3 pad 2: Net-(A1-GND-Pad29) -> Net-(A1-A2)
- C4 pad 1: Net-(A1-A3) -> Net-(A1-GND-Pad29)
- C4 pad 2: Net-(A1-GND-Pad29) -> Net-(A1-A3)
- D1 pad 2: Net-(A1-D4) -> Net-(D1-A)
- D2 pad 2: Net-(A1-D3) -> Net-(D2-A)
- D3 pad 2: Net-(A1-D8) -> Net-(A1-D2)
- D4 pad 2: Net-(A1-D9) -> Net-(A1-D5)
- D5 pad 1: Net-(D5-K) -> Net-(A1-+5V)
- R3 pad 1: Net-(D5-K) -> Net-(A1-+5V)
- S1 pad SH1: Net-(S1A-SHIELD-PadSH1) -> unconnected-(S1A-SHIELD-PadSH1)_1
- S1 pad SH2: Net-(S1A-SHIELD-PadSH1) -> unconnected-(S1A-SHIELD-PadSH1)_3
- S1 pad SH3: Net-(S1A-SHIELD-PadSH1) -> unconnected-(S1A-SHIELD-PadSH1)
- S1 pad SH4: Net-(S1A-SHIELD-PadSH1) -> unconnected-(S1A-SHIELD-PadSH1)_2
- S1 pad VR1_1: Net-(D5-K) -> Net-(A1-+5V)
- S1 pad VR2_1: Net-(D5-K) -> Net-(A1-+5V)
- S2 pad SH1: Net-(S2A-SHIELD-PadSH1) -> unconnected-(S2A-SHIELD-PadSH1)_2
- S2 pad SH2: Net-(S2A-SHIELD-PadSH1) -> unconnected-(S2A-SHIELD-PadSH1)_3
- S2 pad SH3: Net-(S2A-SHIELD-PadSH1) -> unconnected-(S2A-SHIELD-PadSH1)_1
- S2 pad SH4: Net-(S2A-SHIELD-PadSH1) -> unconnected-(S2A-SHIELD-PadSH1)
- SW3 pad 1: unconnected-(SW3-Pad1) -> Net-(A1-GND-Pad29)
- SW3 pad 2: unconnected-(SW3-Pad2) -> Net-(A1-D8)

Commit message: Fixing resistor val.
Parts:
- added R6: 330, Resistor_SMD:R_0805_2012Metric_Pad1.20x1.40mm_HandSolder, F.Cu at (207.9, 49.0)
- added R7: 330, Resistor_SMD:R_0805_2012Metric_Pad1.20x1.40mm_HandSolder, F.Cu at (207.9, 51.9)
- R4, R5: value 300 -> 330
- SW1: value TRIGGER -> TRIGGER_1
- SW10: value DOWN -> DOWN_2
- SW11: value LEFT -> LEFT_2
- SW2: value TRIGGER -> TRIGGER_2
- SW3: value SW_Push -> Calibrate
- SW4: value UP -> UP_1
- SW5: value DOWN -> DOWN_1
- SW6: value LEFT -> LEFT_1
- SW7: value RIGHT -> RIGHT_1
- SW8: value RIGHT -> RIGHT_2
- SW9: value UP -> UP_2
- moved SW11 25.0 mm to (188.5, 72.5)
- moved SW10 16.3 mm to (202.8, 81.8)
- moved SW8 12.6 mm to (214.5, 71.5)
- moved SW9 10.3 mm to (201.5, 64.5)
- moved SW5 4.00 mm to (84.8, 84.5)
- moved SW4 3.75 mm to (84.8, 69.0)
Connections:
- D3 pad 2: Net-(A1-D2) -> Net-(D3-A)
- D4 pad 2: Net-(A1-D5) -> Net-(D4-A)
- J2 pad 7: Net-(J2-Pad7) -> unconnected-(J2-Pad7)
- S2 pad VR1_1: Net-(J2-Pad7) -> Net-(A1-+5V)
- S2 pad VR2_1: Net-(J2-Pad7) -> Net-(A1-+5V)

Commit message: working on PCB layout
Parts:
- moved R4 145.0 mm to (136.0, 56.0)
- moved R5 130.8 mm to (117.0, 66.0)
- moved C1 76.3 mm to (73.0, 44.0)
- moved C2 76.3 mm to (74.0, 51.0)
- moved C3 59.0 mm to (209.0, 44.5)
- moved C4 59.0 mm to (209.0, 47.5)
- moved S1 48.8 mm to (99.0, 58.7)
- moved S2 44.9 mm to (191.4, 58.0)
- moved R6 43.3 mm to (165.0, 43.0)
- moved R7 43.3 mm to (165.0, 46.0)
- moved SW6 41.4 mm to (115.0, 79.5)
- moved SW8 40.8 mm to (174.5, 79.5)
- moved SW5 38.4 mm to (123.0, 87.5)
- moved SW4 38.3 mm to (123.0, 71.5)
- moved SW10 36.7 mm to (166.5, 87.5)
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
Commit message: working on viper PCB layout
Parts:
- A1, J1, J2: moved to B.Cu
- moved SW10 61.1 mm to (121.2, 128.5)
- moved SW11 61.1 mm to (113.2, 120.5)
- moved SW8 61.1 mm to (129.2, 120.5)
- moved SW9 61.1 mm to (121.2, 112.5)
- moved C2 61.0 mm to (108.2, 101.5), turned to -90 degrees
- moved SW4 57.8 mm to (164.0, 112.2)
- moved SW5 57.8 mm to (164.0, 128.2)
- moved SW6 57.8 mm to (156.0, 120.2)
- moved SW7 57.8 mm to (172.0, 120.2)
- moved D1 56.8 mm to (118.5, 93.2), turned to -90 degrees
- moved C4 53.8 mm to (201.5, 100.8), turned to -90 degrees
- moved C1 51.3 mm to (94.7, 90.5)
- moved R6 50.5 mm to (158.2, 93.0)
- moved SW2 50.3 mm to (197.8, 79.2), turned to -90 degrees
- moved C3 50.0 mm to (187.2, 89.5)
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Other:
- board size 168 x 102 mm -> 141 x 68.5 mm

Commit message: working on viper PCB layout
Parts:
- moved SW3 9.25 mm to (88.8, 78.2)
- moved C3 6.22 mm to (193.3, 90.8)
- moved S2 6.14 mm to (194.5, 103.0)
- moved R7 5.26 mm to (158.8, 92.2)
- moved C4 5.19 mm to (206.6, 101.8)
- moved SW1 5.00 mm to (99.8, 78.5), turned to 0 degrees
- moved SW4 4.26 mm to (168.2, 112.5)
- moved SW5 4.26 mm to (168.2, 128.5)
- moved SW6 4.26 mm to (160.2, 120.5)
- moved SW7 4.26 mm to (176.2, 120.5)
- moved SW2 3.50 mm to (194.2, 79.2), turned to 180 degrees
- moved D3 3.09 mm to (173.8, 96.0)
- moved R6 3.04 mm to (158.8, 96.0)
- moved SW10 3.00 mm to (118.2, 128.5)
- moved SW11 3.00 mm to (110.2, 120.5)
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Routing:
- net Net-(A1-GND-Pad29): track 0.00 -> 111.0 mm
- net Net-(D4-A): track 0.00 -> 3.92 mm
- net Net-(D3-A): track 0.00 -> 3.92 mm
- net Net-(A1-A2): track 0.00 -> 3.57 mm
- net Net-(A1-A3): track 0.00 -> 3.41 mm
- net Net-(A1-A0): track 0.00 -> 3.35 mm
- net Net-(A1-A1): track 0.00 -> 3.33 mm

Commit message: working on viper PCB layout
Parts:
- C1, C2, C3, R1, R4, R5: moved to B.Cu
- moved SW4 77.1 mm to (93.8, 92.8)
- moved SW5 77.1 mm to (93.8, 108.8)
- moved SW6 77.1 mm to (85.8, 100.8)
- moved SW7 77.1 mm to (101.8, 100.8)
- moved SW10 76.1 mm to (191.8, 108.8)
- moved SW11 76.1 mm to (183.8, 100.8)
- moved SW8 76.1 mm to (199.8, 100.8)
- moved SW9 76.1 mm to (191.8, 92.8)
- moved C3 30.1 mm to (169.8, 109.5)
- moved C4 30.1 mm to (183.1, 120.5)
- moved S2 30.1 mm to (171.0, 121.7)
- moved C1 29.8 mm to (120.0, 109.8)
- moved S1 29.6 mm to (121.0, 121.7)
- moved C2 29.4 mm to (132.8, 120.5)
- moved F1 17.5 mm to (127.0, 76.0)
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Routing:
- net Net-(A1-GND-Pad29): track 111.0 -> 378.3 mm
- net Net-(A1-+5V): track 0.00 -> 123.5 mm
- net Net-(A1-D8): track 0.00 -> 53.8 mm
- net Net-(A1-A3): track 3.41 -> 56.7 mm
- net Net-(J1-Pad2): track 0.00 -> 47.8 mm
- net Net-(A1-A1): track 3.33 -> 50.6 mm
- net Net-(A1-A0): track 3.35 -> 49.2 mm
- net Net-(J1-Pad3): track 0.00 -> 43.7 mm
- net Net-(J1-Pad1): track 0.00 -> 43.6 mm
- net Net-(J2-Pad4): track 0.00 -> 43.5 mm
- net Net-(J2-Pad2): track 0.00 -> 40.2 mm
- net Net-(J2-Pad3): track 0.00 -> 32.7 mm
- net Net-(A1-A2): track 3.57 -> 34.4 mm
- net Net-(J1-Pad4): track 0.00 -> 29.2 mm
- net Net-(J1-Pad6): track 0.00 -> 24.8 mm
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
Commit message: working on viper PCB layout
Parts:
- added REF**: MountingHole_3.2mm_M3, MountingHole:MountingHole_3.2mm_M3, F.Cu at (80.0, 76.8)
- added REF**: MountingHole_3.2mm_M3, MountingHole:MountingHole_3.2mm_M3, F.Cu at (210.0, 76.8)
- added REF**: MountingHole_3.2mm_M3, MountingHole:MountingHole_3.2mm_M3, F.Cu at (80.0, 134.2)
- added REF**: MountingHole_3.2mm_M3, MountingHole:MountingHole_3.2mm_M3, F.Cu at (210.0, 134.2)
